File: hardware/decoder/decoder.kicad_sch (KiCad schematic)
At the start: 50 parts, among them J1 Conn_02x32_Counter_Clockwise, J2 DC37_Receptacle, U1 4050, U10 MC68B09, U11 74LS241, U12 AM2732DC, U13 74LS02, U14 74LS74, U15 74LS27, U16 HM6116LP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

Commit message: routing done
Connections:
- net COMP_Q0: no longer J1.2 (Pin_2)
- net COMP_Q1: no longer J1.3 (Pin_3)
- net COMP_Q2: no longer J1.4 (Pin_4)
- net COMP_Q3: no longer J1.5 (Pin_5)
- net COMP_Q4: no longer J1.6 (Pin_6)
- net COMP_Q5: no longer J1.7 (Pin_7)
- net COMP_Q6: no longer J1.8 (Pin_8)
- net COMP_Q7: no longer J1.9 (Pin_9)
- net COMP_EQ renamed ADD_MATCH
- net CON16 renamed DISCRIM_OUT
- new net CARD_A0: J1.2 (Pin_2)
- new net CARD_A1: J1.3 (Pin_3)
- new net CARD_A2: J1.4 (Pin_4)
- new net CARD_A3: J1.5 (Pin_5)
- new net CARD_A4: J1.6 (Pin_6)
- new net CARD_A5: J1.7 (Pin_7)
- new net CARD_A6: J1.8 (Pin_8)
- new net CARD_A7: J1.9 (Pin_9)
Changed lines of the file:
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@@
 		)
 	)
-	(label "COMP_Q1"
-		(at 742.95 276.86 0)
-		(fields_autoplaced yes)
-		(effects
-			(font
-				(size 1.27 1.27)
-			)
-			(justify left bottom)
-		)
-	)
 	(label "FIFO_EXT_A1"
 		(at 798.83 274.32 180)
@@
 		)
 	)
-	(label "COMP_Q6"
-		(at 742.95 289.56 0)
-		(fields_autoplaced yes)
-		(effects
-			(font
-				(size 1.27 1.27)
-			)
-			(justify left bottom)
-		)
-	)
 	(label "RB_A1"
 		(at 121.92 363.22 0)
@@
 		)
 	)
-	(label "CON16"
+	(label "DISCRIM_OUT"
 		(at 490.22 505.46 0)
 		(fields_autoplaced yes)
@@
 		)
 	)
-	(label "COMP_EQ"
+	(label "ADD_MATCH"
 		(at 622.3 96.52 0)
 		(fields_autoplaced yes)
@@
 		)
 	)
+	(label "CARD_A2"
+		(at 742.95 279.4 0)
+		(fields_autoplaced yes)
+		(effects
+			(font
+				(size 1.27 1.27)
+			)
+			(justify left bottom)
+		)
+	)
 	(label "~{FIFO_CS}"
 		(at 467.36 487.68 180)
@@
 		)
 	)
-	(label "COMP_Q0"
-		(at 742.95 274.32 0)
-		(fields_autoplaced yes)
-		(effects
-			(font
-				(size 1.27 1.27)
-			)
-			(justify left bottom)
-		)
-	)
 	(label "~{WE}"
 		(at 607.06 492.76 180)
@@
 		)
 	)
-	(label "CON16"
+	(label "DISCRIM_OUT"
 		(at 742.95 309.88 0)
 		(fields_autoplaced yes)
@@
 		)
 	)
-	(label "COMP_Q2"
-		(at 742.95 279.4 0)
-		(fields_autoplaced yes)
-		(effects
-			(font
-				(size 1.27 1.27)
-			)
-			(justify left bottom)
-		)
-	)
 	(label "DC37_16"
 		(at 49.53 280.67 180)
@@
 		)
 	)
+	(label "CARD_A7"
+		(at 742.95 292.1 0)
+		(fields_autoplaced yes)
+		(effects
+			(font
+				(size 1.27 1.27)
+			)
+			(justify left bottom)
+		)
+	)
 	(label "RB_B6"
 		(at 121.92 421.64 0)
@@
 		)
 	)
+	(label "CARD_A4"
+		(at 742.95 284.48 0)
+		(fields_autoplaced yes)
+		(effects
+			(font
+				(size 1.27 1.27)
+			)
+			(justify left bottom)
+		)
+	)
 	(label "DC37_35"
 		(at 64.77 306.07 0)
@@
 		)
 	)
-	(label "COMP_Q3"
-		(at 742.95 281.94 0)
-		(fields_autoplaced yes)
-		(effects
-			(font
-				(size 1.27 1.27)
-			)
-			(justify left bottom)
-		)
-	)
 	(label "RB_A7"
 		(at 102.87 387.35 180)
@@
 		)
 	)
-	(label "COMP_EQ"
+	(label "ADD_MATCH"
 		(at 774.7 203.2 180)
 		(fields_autoplaced yes)
@@
 		)
 	)
-	(label "COMP_Q7"
-		(at 742.95 292.1 0)
+	(label "DC37_6"
+		(at 49.53 331.47 180)
 		(fields_autoplaced yes)
 		(effects
@@
 				(size 1.27 1.27)
 			)
-			(justify left bottom)
+			(justify right bottom)
 		)
 	)
-	(label "DC37_6"
-		(at 49.53 331.47 180)
+	(label "CARD_A3"
+		(at 742.95 281.94 0)
 		(fields_autoplaced yes)
 		(effects
@@
 				(size 1.27 1.27)
 			)
-			(justify right bottom)
+			(justify left bottom)
 		)
 	)
@@
 		)
 	)
-	(label "COMP_Q5"
-		(at 742.95 287.02 0)
-		(fields_autoplaced yes)
-		(effects
-			(font
-				(size 1.27 1.27)
-			)
-			(justify left bottom)
-		)
-	)
 	(label "DC37_22"
 		(at 49.53 344.17 180)
@@
 		)
 	)
-	(label "COMP_Q4"
-		(at 742.95 284.48 0)
+	(label "RA_A2"
+		(at 121.92 203.2 0)
 		(fields_autoplaced yes)
 		(effects
@@
 		)
 	)
-	(label "RA_A2"
-		(at 121.92 203.2 0)
+	(label "DC37_7"
+		(at 64.77 336.55 0)
 		(fields_autoplaced yes)
 		(effects
@@
 		)
 	)
-	(label "DC37_7"
-		(at 64.77 336.55 0)
+	(label "A9"
+		(at 347.98 495.3 0)
 		(fields_autoplaced yes)
 		(effects
@@
 		)
 	)
-	(label "A9"
-		(at 347.98 495.3 0)
+	(label "CARD_A6"
+		(at 742.95 289.56 0)
 		(fields_autoplaced yes)
 		(effects
@@
 		)
 	)
+	(label "CARD_A5"
+		(at 742.95 287.02 0)
+		(fields_autoplaced yes)
+		(effects
+			(font
+				(size 1.27 1.27)
+			)
+			(justify left bottom)
+		)
+	)
 	(label "A10"
 		(at 276.86 497.84 0)
@@
 		)
 	)
+	(label "CARD_A0"
+		(at 742.95 274.32 0)
+		(fields_autoplaced yes)
+		(effects
+			(font
+				(size 1.27 1.27)
+			)
+			(justify left bottom)
+		)
+	)
 	(label "DC37_1"
 		(at 49.53 356.87 180)
@@
 		(fields_autoplaced yes)
 		(effects
+			(font
+				(size 1.27 1.27)
+			)
+			(justify left bottom)
+		)
+	)
+	(label "CARD_A1"
+		(at 742.95 276.86 0)
+		(fields_autoplaced yes)
+		(effects
