File: hardware/decoder_baseboard/decoder_baseboard.kicad_pcb (KiCad board)
At the start: 2 copper layers, 50.6 x 129 mm, 11 parts, among them J2 USB_C_Receptacle_USB2.0, U1 SN74AVC8T245PW, U2 PicoW

Commit message: Some routing done
Parts:
- removed J2: USB_C_Receptacle_USB2.0, Connector_USB:USB_C_Receptacle_XKB_U262-16XN-4BVC11
- added C10: 100n, Capacitor_SMD:C_0603_1608Metric, F.Cu at (198.5, 90.9)
- added C11: 10u, Capacitor_SMD:C_0603_1608Metric, B.Cu at (205.1, 84.5)
- added C2: 100n, Capacitor_SMD:C_0603_1608Metric, B.Cu at (138.5, 99.5)
- added C4: 100n, Capacitor_SMD:C_0603_1608Metric, F.Cu at (204.5, 118.5)
- added C5: 100n, Capacitor_SMD:C_0603_1608Metric, B.Cu at (222.5, 124.7)
- added C6: 100n, Capacitor_SMD:C_0603_1608Metric, F.Cu at (192.5, 106.4)
- added C7: 10u, Capacitor_SMD:C_0603_1608Metric, B.Cu at (222.5, 121.7)
- added C8: 10u, Capacitor_SMD:C_0603_1608Metric, B.Cu at (211.5, 121.7)
- added C9: 100n, Capacitor_SMD:C_0603_1608Metric, B.Cu at (211.5, 124.7)
- added D1: LED FILAMENT, decoder:Con_01x02_2.54_SMD, B.Cu at (214.2, 34.8)
- added D2: BAV99, Package_TO_SOT_SMD:SOT-23, B.Cu at (126.0, 102.8)
- added J1: Conn_02x32_Odd_Even, Connector_PinSocket_2.54mm:PinSocket_2x32_P2.54mm_Vertical_SMD, B.Cu at (217.2, 86.4)
- added J3: USB4800, Connector_USB:USB_C_Receptacle_XKB_U262-16XN-4BVC11, B.Cu at (198.5, 84.8)
- added JP1: SolderJumper_3_Bridged12, Jumper:SolderJumper-3_P1.3mm_Bridged2Bar12_Pad1.0x1.5mm, F.Cu at (210.5, 39.8)
- added JP2: SolderJumper_3_Bridged12, Jumper:SolderJumper-3_P1.3mm_Bridged2Bar12_Pad1.0x1.5mm, F.Cu at (207.1, 39.8)
- added JP3: SolderJumper_3_Bridged12, Jumper:SolderJumper-3_P1.3mm_Bridged2Bar12_Pad1.0x1.5mm, F.Cu at (203.6, 39.8)
- added JP4: SolderJumper_3_Bridged12, Jumper:SolderJumper-3_P1.3mm_Bridged2Bar12_Pad1.0x1.5mm, F.Cu at (200.2, 39.8)
- added JP5: SolderJumper_3_Bridged12, Jumper:SolderJumper-3_P1.3mm_Bridged2Bar12_Pad1.0x1.5mm, F.Cu at (196.8, 39.8)
- added JP6: SolderJumper_3_Bridged12, Jumper:SolderJumper-3_P1.3mm_Bridged2Bar12_Pad1.0x1.5mm, F.Cu at (193.4, 39.8)
- added JP7: SolderJumper_3_Bridged12, Jumper:SolderJumper-3_P1.3mm_Bridged2Bar12_Pad1.0x1.5mm, F.Cu at (189.9, 39.8)
- added JP8: SolderJumper_3_Bridged12, Jumper:SolderJumper-3_P1.3mm_Bridged2Bar12_Pad1.0x1.5mm, F.Cu at (186.5, 39.8)
- added LS1: PKMCS0909E, Buzzer_Beeper:Buzzer_Murata_PKMCS0909E, F.Cu at (198.5, 127.5)
- added Q1: BSS138, Package_TO_SOT_SMD:SOT-23, B.Cu at (215.4, 39.1)
- added Q2: BSS138, Package_TO_SOT_SMD:SOT-23, F.Cu at (199.4, 134.2)
- added R1: 5k1, Resistor_SMD:R_0603_1608Metric, B.Cu at (201.8, 78.9)
- added R2: 5k1, Resistor_SMD:R_0603_1608Metric, B.Cu at (195.2, 78.9)
- added R3: 22k, Resistor_SMD:R_0603_1608Metric, B.Cu at (130.5, 99.5)
- added R4: 33k, Resistor_SMD:R_0603_1608Metric, B.Cu at (130.5, 102.0)
- added R5: 10k, Resistor_SMD:R_0603_1608Metric, B.Cu at (115.2, 99.2)
- added R6: 33, Resistor_SMD:R_0603_1608Metric, B.Cu at (212.9, 39.1)
- added R7: 10k, Resistor_SMD:R_0603_1608Metric, B.Cu at (215.5, 42.1)
- added R8: 10k, Resistor_SMD:R_0603_1608Metric, F.Cu at (202.5, 134.2)
- added U3: USBLC6-2SC6, Package_TO_SOT_SMD:SOT-23-6, B.Cu at (198.5, 77.0)
- added U4: LIS2DW12, Package_LGA:LGA-12_2x2mm_P0.5mm, F.Cu at (198.5, 94.0)
- added U6: SN74HCS244, Package_SO:TSSOP-20_4.4x6.5mm_P0.65mm, F.Cu at (198.5, 103.5)
- C1: value 1u -> 10u; moved to B.Cu
- C3: value 10u -> 100n
- R10: value 5k1 -> 1k
- R9: value 5k1 -> 100
- U1: value SN74AVC8T245PW -> SN74LXC8T245
- moved R10 134.7 mm to (196.4, 134.2), turned to -90 degrees
- moved R9 134.6 mm to (194.5, 134.2), turned to 90 degrees
- moved C3 125.7 mm to (192.5, 118.5), turned to 180 degrees
- moved U1 122.8 mm to (198.5, 114.9), turned to 180 degrees
- moved C1 112.1 mm to (191.9, 84.5), turned to -90 degrees
Connections:
- C1 pad 1: GND -> +5V
- C1 pad 2: +5V -> GND
- R10 pad 1: +5V -> Net-(LS1-Pad1)
- R9 pad 1: Net-(J2-CC1) -> +5V
- R9 pad 2: +5V -> Net-(LS1-Pad1)
- U1 pad 1: unconnected-(U1-VCCA-Pad1) -> +3V3
- U1 pad 11: Net-(U1-GND-Pad11) -> GND
- U1 pad 12: Net-(U1-GND-Pad11) -> GND
- U1 pad 13: Net-(U1-GND-Pad11) -> GND
- U1 pad 14: unconnected-(U1-B8-Pad14) -> /FIFO_EXT_D0
- U1 pad 15: unconnected-(U1-B7-Pad15) -> /FIFO_EXT_D4
- U1 pad 16: unconnected-(U1-B6-Pad16) -> /FIFO_EXT_D1
- U1 pad 17: unconnected-(U1-B5-Pad17) -> /FIFO_EXT_D5
- U1 pad 18: unconnected-(U1-B4-Pad18) -> /FIFO_EXT_D2
- U1 pad 19: unconnected-(U1-B3-Pad19) -> /FIFO_EXT_D6
- U1 pad 20: unconnected-(U1-B2-Pad20) -> /FIFO_EXT_D3
- U1 pad 21: unconnected-(U1-B1-Pad21) -> /FIFO_EXT_D7
- U1 pad 22: unconnected-(U1-~{OE}-Pad22) -> Net-(U1-~{OE})
- U1 pad 23: unconnected-(U1-VCCB-Pad23) -> +5V
- U1 pad 24: unconnected-(U1-VCCB-Pad24) -> +5V
- U2 pad 1: /CON_D0 -> unconnected-(U2-GPIO0-Pad1)
- U2 pad 10: /CON_D7 -> unconnected-(U2-GPIO7-Pad10)
- U2 pad 2: /CON_D1 -> unconnected-(U2-GPIO1-Pad2)
- U2 pad 36: unconnected-(U2-3V3-Pad36) -> +3V3
- U2 pad 39: unconnected-(U2-VSYS-Pad39) -> +5V
- U2 pad 4: /CON_D2 -> unconnected-(U2-GPIO2-Pad4)
- U2 pad 5: /CON_D3 -> unconnected-(U2-GPIO3-Pad5)
- U2 pad 6: /CON_D4 -> unconnected-(U2-GPIO4-Pad6)
- U2 pad 7: /CON_D5 -> unconnected-(U2-GPIO5-Pad7)
- U2 pad 9: /CON_D6 -> unconnected-(U2-GPIO6-Pad9)
Routing:
- net +5V: track 0.00 -> 257.5 mm, vias 0 -> 3
- net /CARD_A7: track 0.00 -> 54.5 mm
- net /CARD_A6: track 0.00 -> 47.9 mm
- net /CARD_A5: track 0.00 -> 42.4 mm
- net /CARD_A4: track 0.00 -> 36.9 mm
- net /FIFO_EXT_D0: track 0.00 -> 32.9 mm
- net /FIFO_EXT_D2: track 0.00 -> 31.2 mm
- net /CARD_A3: track 0.00 -> 30.9 mm
- net /FIFO_EXT_D1: track 0.00 -> 29.3 mm
- net /FIFO_EXT_D3: track 0.00 -> 28.3 mm
- net +3V3: track 0.00 -> 25.5 mm, vias 0 -> 5
- net /CARD_A2: track 0.00 -> 25.1 mm
- net /FIFO_EXT_D4: track 0.00 -> 24.6 mm
- net /FIFO_EXT_D7: track 0.00 -> 23.5 mm
- net /FIFO_EXT_D5: track 0.00 -> 23.2 mm
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- added copper zone on B.Cu, net +5V
- added copper zone on B.Cu, net GND
- added copper zone on F.Cu, net GND
Other:
- board text added: "A0"
- board text added: "A1"
- board text added: "A2"
- board text added: "A3"
- board text added: "A4"
- board text added: "A5"
- board text added: "A6"
- board text added: "A7"

Commit message: routing done
Parts:
- removed C2: 100n, Capacitor_SMD:C_0603_1608Metric
- removed D2: BAV99, Package_TO_SOT_SMD:SOT-23
- removed R3: 22k, Resistor_SMD:R_0603_1608Metric
- removed R4: 33k, Resistor_SMD:R_0603_1608Metric
- added C12: 10u, Capacitor_SMD:C_0603_1608Metric, B.Cu at (211.1, 74.4)
- added C13: 10u, Capacitor_SMD:C_0603_1608Metric, B.Cu at (193.3, 74.4)
- Q2, R10, R8, R9: moved to B.Cu
- moved R5 84.2 mm to (198.5, 111.3), turned to -90 degrees
- moved C3 13.9 mm to (204.5, 111.5), turned to 0 degrees
- moved C4 13.9 mm to (192.5, 111.5), turned to 180 degrees
- moved C6 13.2 mm to (204.5, 100.8), turned to 0 degrees
- moved R8 8.81 mm to (194.5, 130.4)
- moved R9 8.81 mm to (202.5, 130.4), turned to -90 degrees
- moved R10 5.64 mm to (200.6, 130.4), turned to 90 degrees
- moved Q2 4.15 mm to (197.6, 130.4), turned to 0 degrees
- moved JP1 4.00 mm to (206.5, 39.8)
- moved JP8 4.00 mm to (190.5, 39.8)
- moved JP7 2.86 mm to (192.8, 39.8)
- moved JP2 2.86 mm to (204.2, 39.8)
- moved JP6 1.71 mm to (195.1, 39.8)
- moved JP3 1.71 mm to (201.9, 39.8)
- moved R6 1.02 mm to (212.9, 38.1)
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Connections:
- J1 pad 60: +12V -> unconnected-(J1-Pin_60-Pad60)
- R5 pad 2: Net-(U1-~{OE}) -> /TRCVR_~{OE}
- U1 pad 10: unconnected-(U1-A8-Pad10) -> /FIFO_D7_3V3
- U1 pad 14: /FIFO_EXT_D0 -> /FIFO_EXT_D7
- U1 pad 15: /FIFO_EXT_D4 -> /FIFO_EXT_D3
- U1 pad 16: /FIFO_EXT_D1 -> /FIFO_EXT_D6
- U1 pad 17: /FIFO_EXT_D5 -> /FIFO_EXT_D2
- U1 pad 18: /FIFO_EXT_D2 -> /FIFO_EXT_D5
- U1 pad 19: /FIFO_EXT_D6 -> /FIFO_EXT_D1
- U1 pad 2: unconnected-(U1-DIR-Pad2) -> /TRCVR_DIR
- U1 pad 20: /FIFO_EXT_D3 -> /FIFO_EXT_D4
- U1 pad 21: /FIFO_EXT_D7 -> /FIFO_EXT_D0
- U1 pad 22: Net-(U1-~{OE}) -> /TRCVR_~{OE}
- U1 pad 3: unconnected-(U1-A1-Pad3) -> /FIFO_D0_3V3
- U1 pad 4: unconnected-(U1-A2-Pad4) -> /FIFO_D4_3V3
- U1 pad 5: unconnected-(U1-A3-Pad5) -> /FIFO_D1_3V3
- U1 pad 6: unconnected-(U1-A4-Pad6) -> /FIFO_D5_3V3
- U1 pad 7: unconnected-(U1-A5-Pad7) -> /FIFO_D2_3V3
- U1 pad 8: unconnected-(U1-A6-Pad8) -> /FIFO_D6_3V3
- U1 pad 9: unconnected-(U1-A7-Pad9) -> /FIFO_D3_3V3
- U2 pad 10: unconnected-(U2-GPIO7-Pad10) -> /TRCVR_DIR
- U2 pad 11: unconnected-(U2-GPIO8-Pad11) -> /FIFO_D0_3V3
- U2 pad 12: unconnected-(U2-GPIO9-Pad12) -> /FIFO_D4_3V3
- U2 pad 14: unconnected-(U2-GPIO10-Pad14) -> /FIFO_D1_3V3
- U2 pad 15: unconnected-(U2-GPIO11-Pad15) -> /FIFO_D5_3V3
- U2 pad 16: unconnected-(U2-GPIO12-Pad16) -> /FIFO_D2_3V3
- U2 pad 17: unconnected-(U2-GPIO13-Pad17) -> /FIFO_D6_3V3
- U2 pad 19: unconnected-(U2-GPIO14-Pad19) -> /FIFO_D3_3V3
- U2 pad 2: unconnected-(U2-GPIO1-Pad2) -> /FIFO_EN_3V3
- U2 pad 20: unconnected-(U2-GPIO15-Pad20) -> /FIFO_D7_3V3
- U2 pad 24: unconnected-(U2-GPIO18-Pad24) -> /ACCEL_SDA
- U2 pad 25: unconnected-(U2-GPIO19-Pad25) -> /ACCEL_SCL
- U2 pad 26: unconnected-(U2-GPIO20-Pad26) -> /ACCEL_INT1
- U2 pad 27: unconnected-(U2-GPIO21-Pad27) -> /ACCEL_INT2
- U2 pad 29: unconnected-(U2-GPIO22-Pad29) -> /ACCEL_~{CS}
- U2 pad 4: unconnected-(U2-GPIO2-Pad4) -> /FIFO_R/~{W}_3V3
- U2 pad 5: unconnected-(U2-GPIO3-Pad5) -> /~{RESET}_3V3
- U2 pad 6: unconnected-(U2-GPIO4-Pad6) -> /FIFO_A1_3V3
- U2 pad 7: unconnected-(U2-GPIO5-Pad7) -> /FIFO_A0_3V3
- U2 pad 9: unconnected-(U2-GPIO6-Pad9) -> /TRCVR_~{OE}
- U6 pad 1: unconnected-(U6-1OE-Pad1) -> GND
- U6 pad 11: unconnected-(U6-2A3-Pad11) -> GND
- U6 pad 13: unconnected-(U6-2A2-Pad13) -> GND
- U6 pad 14: /~{RESET} -> /FIFO_EXT_EN
- U6 pad 15: unconnected-(U6-2A1-Pad15) -> GND
- U6 pad 16: /FIFO_EXT_R/~{W} -> /~{RESET}
- U6 pad 17: unconnected-(U6-2A0-Pad17) -> /FIFO_A0_3V3
- U6 pad 18: /FIFO_EXT_EN -> /FIFO_EXT_R/~{W}
- U6 pad 19: unconnected-(U6-2OE-Pad19) -> GND
- U6 pad 2: unconnected-(U6-1A0-Pad2) -> /FIFO_EN_3V3
- U6 pad 4: unconnected-(U6-1A1-Pad4) -> /FIFO_R/~{W}_3V3
- U6 pad 6: unconnected-(U6-1A2-Pad6) -> /~{RESET}_3V3
- U6 pad 8: unconnected-(U6-1A3-Pad8) -> /FIFO_A1_3V3
Routing:
- net /FIFO_D7_3V3: track 0.00 -> 115.9 mm, vias 0 -> 1
- net /FIFO_D3_3V3: track 0.00 -> 112.1 mm, vias 0 -> 1
- net /FIFO_D6_3V3: track 0.00 -> 105.7 mm, vias 0 -> 1
- net /FIFO_D2_3V3: track 0.00 -> 101.9 mm, vias 0 -> 1
- net /FIFO_D5_3V3: track 0.00 -> 98.1 mm, vias 0 -> 1
- net /ACCEL_SDA: track 0.00 -> 96.8 mm, vias 0 -> 1
- net /FIFO_D1_3V3: track 0.00 -> 94.2 mm, vias 0 -> 1
- net /FIFO_D4_3V3: track 0.00 -> 87.9 mm, vias 0 -> 1
- net /TRCVR_DIR: track 0.00 -> 84.7 mm, vias 0 -> 1
- net /ACCEL_SCL: track 0.00 -> 84.7 mm, vias 0 -> 1
- net /FIFO_D0_3V3: track 0.00 -> 84.1 mm, vias 0 -> 1
- net /TRCVR_~{OE}: track 0.00 -> 83.9 mm, vias 0 -> 2
- net /ACCEL_~{CS}: track 0.00 -> 83.5 mm, vias 0 -> 1
- net /FIFO_A0_3V3: track 0.00 -> 82.3 mm, vias 0 -> 1
- net /FIFO_EXT_A1: track 0.00 -> 80.7 mm, vias 0 -> 1
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Other:
- board text added: "+"
- board text added: "-"
- board text added: "H"
- board text added: "L"
