File: hardware/decoder_baseboard/decoder_baseboard.kicad_pcb (KiCad board)
At the start: 2 copper layers, 50.6 x 129 mm, 43 parts, among them J1 Conn_02x32_Odd_Even, J3 USB4800, Q1 BSS138, Q2 BSS138, U1 SN74LXC8T245, U2 PicoW, U3 USBLC6-2SC6, U4 LIS2DW12, U6 SN74HCS244

Commit message: Got FW working
Parts:
- J3: footprint Connector_USB:USB_C_Receptacle_XKB_U262-16XN-4BVC11 -> decoder:USB_C_Receptacle_GCT_USB4800
