File: hardware/decoder_baseboard/_autosave-decoder_baseboard.kicad_sch (KiCad schematic)
At the start: 43 parts, among them J1 Conn_02x32_Odd_Even, J3 USB4800, Q1 BSS138, Q2 BSS138, U1 SN74LXC8T245, U2 PicoW, U3 USBLC6-2SC6, U4 LIS2DW12, U6 SN74HCS244

Commit message: routing done
Connections:
- net BACKLIGHT_PWM: now also U2.21 (GPIO16)
- no-connect marks 55 -> 54
Changed lines of the file:
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@@
-	)
-	(no_connect
-		(at 363.22 215.9)
 	)
 	(no_connect
@@
 		(pts
 			(xy 45.72 67.31) (xy 45.72 74.93)
+		)
+		(stroke
+			(width 0)
+			(type default)
+		)
+	)
+	(wire
+		(pts
+			(xy 363.22 215.9) (xy 381 215.9)
 		)
 		(stroke
@@
 		)
 	)
+	(label "BACKLIGHT_PWM"
+		(at 381 215.9 180)
+		(fields_autoplaced yes)
+		(effects
+			(font
+				(size 1.27 1.27)
+			)
+			(justify right bottom)
+		)
+	)

Commit message: routing done
Parts:
- H1, H2, H3, H4: footprint MountingHole:MountingHole_2.2mm_M2_DIN965_Pad -> MountingHole:MountingHole_2.5mm
Changed lines of the file:
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@@
 			)
 		)
-		(property "Footprint" "MountingHole:MountingHole_2.2mm_M2_DIN965_Pad"
+		(property "Footprint" "MountingHole:MountingHole_2.5mm"
 			(at 290.83 273.05 0)
 			(effects
@@
 			)
 		)
-		(property "Footprint" "MountingHole:MountingHole_2.2mm_M2_DIN965_Pad"
+		(property "Footprint" "MountingHole:MountingHole_2.5mm"
 			(at 281.94 273.05 0)
 			(effects
@@
 			)
 		)
-		(property "Footprint" "MountingHole:MountingHole_2.2mm_M2_DIN965_Pad"
+		(property "Footprint" "MountingHole:MountingHole_2.5mm"
 			(at 290.83 279.4 0)
 			(effects
@@
 			)
 		)
-		(property "Footprint" "MountingHole:MountingHole_2.2mm_M2_DIN965_Pad"
+		(property "Footprint" "MountingHole:MountingHole_2.5mm"
 			(at 281.94 279.4 0)
 			(effects
