File: hardware/decoder_baseboard/decoder_baseboard-rounded.kicad_pcb (KiCad board)
At the start: 2 copper layers, 50.6 x 129 mm, 43 parts, among them J1 Conn_02x32_Odd_Even, J3 USB4800, Q1 BSS138, Q2 BSS138, U1 SN74LXC8T245, U2 PicoW, U3 USBLC6-2SC6, U4 LIS2DW12, U6 SN74HCS244

Commit message: routing done
Routing:
- net /FIFO_A1_3V3: track 59.4 -> 61.3 mm
- net /FIFO_D7_3V3: track 114.0 -> 115.9 mm
- net /FIFO_D3_3V3: track 110.5 -> 112.1 mm
- net /FIFO_EXT_D7: track 23.0 -> 24.4 mm
- net /FIFO_D6_3V3: track 104.4 -> 105.7 mm
- net /~{RESET}_3V3: track 55.5 -> 56.8 mm
- net /FIFO_EXT_D3: track 25.1 -> 26.3 mm
- net /FIFO_D2_3V3: track 100.8 -> 101.9 mm
- net /FIFO_EXT_D6: track 24.8 -> 25.7 mm
- net /FIFO_D5_3V3: track 97.3 -> 98.1 mm
- net /FIFO_EXT_D2: track 26.9 -> 27.7 mm
- net /FIFO_R/~{W}_3V3: track 51.7 -> 52.4 mm
- net /FIFO_EXT_R/~{W}: track 34.5 -> 35.2 mm
- net /ACCEL_SDA: track 96.2 -> 96.8 mm
- net /FIFO_EXT_D5: track 26.5 -> 27.1 mm
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
Commit message: finished rounded version
Routing:
- net +5V: track 223.0 -> 225.5 mm
- net GND: track 3.48 -> 1.25 mm, vias 37 -> 431
- net /FIFO_A1_3V3: track 61.3 -> 59.2 mm
- net /FIFO_D7_3V3: track 115.9 -> 113.8 mm
- net /FIFO_D3_3V3: track 112.1 -> 110.3 mm
- net /FIFO_EXT_D7: track 24.4 -> 22.7 mm
- net /FIFO_D6_3V3: track 105.7 -> 104.2 mm
- net /~{RESET}_3V3: track 56.8 -> 55.3 mm
- net /FIFO_EXT_D3: track 26.3 -> 24.9 mm
- net /FIFO_D2_3V3: track 101.9 -> 100.6 mm
- net /FIFO_EXT_D6: track 25.7 -> 24.5 mm
- net /ACCEL_SDA: track 96.8 -> 95.6 mm
- net /FIFO_EXT_D2: track 27.7 -> 26.7 mm
- net /FIFO_D5_3V3: track 98.1 -> 97.1 mm
- net /FIFO_EXT_R/~{W}: track 35.2 -> 34.2 mm
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
Commit message: Sync
Other:
- board text added: "JLCJLCJLCJLC"
