File: hardware/decoder_baseboard/decoder_baseboard.kicad_sch (KiCad schematic)
At the start: 43 parts, among them J1 Conn_02x32_Odd_Even, J3 USB4800, Q1 BSS138, Q2 BSS138, U1 SN74LXC8T245, U2 PicoW, U3 USBLC6-2SC6, U4 LIS2DW12, U6 SN74HCS244

Commit message: sync
Parts:
- H1, H2, H3, H4: footprint MountingHole:MountingHole_2.2mm_M2_DIN965_Pad -> MountingHole:MountingHole_2.5mm
Connections:
- net BACKLIGHT_PWM: now also U2.21 (GPIO16)
- no-connect marks 55 -> 54
Changed lines of the file:
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@@
 	)
 	(no_connect
-		(at 363.22 215.9)
-	)
-	(no_connect
 		(at 60.96 157.48)
 	)
@@
 	(wire
 		(pts
+			(xy 363.22 215.9) (xy 381 215.9)
+		)
+		(stroke
+			(width 0)
+			(type default)
+		)
+	)
+	(wire
+		(pts
 			(xy 45.72 226.06) (xy 45.72 147.32)
 		)
@@
 		)
 	)
+	(label "BACKLIGHT_PWM"
+		(at 381 215.9 180)
+		(fields_autoplaced yes)
+		(effects
+			(font
+				(size 1.27 1.27)
+			)
+			(justify right bottom)
+		)
+	)
 	(label "ACCEL_SCL"
 		(at 381 205.74 180)
@@
 			)
 		)
-		(property "Footprint" "MountingHole:MountingHole_2.2mm_M2_DIN965_Pad"
+		(property "Footprint" "MountingHole:MountingHole_2.5mm"
 			(at 290.83 273.05 0)
 			(effects
@@
 			)
 		)
-		(property "Footprint" "MountingHole:MountingHole_2.2mm_M2_DIN965_Pad"
+		(property "Footprint" "MountingHole:MountingHole_2.5mm"
 			(at 281.94 273.05 0)
 			(effects
@@
 			)
 		)
-		(property "Footprint" "MountingHole:MountingHole_2.2mm_M2_DIN965_Pad"
+		(property "Footprint" "MountingHole:MountingHole_2.5mm"
 			(at 290.83 279.4 0)
 			(effects
@@
 			)
 		)
-		(property "Footprint" "MountingHole:MountingHole_2.2mm_M2_DIN965_Pad"
+		(property "Footprint" "MountingHole:MountingHole_2.5mm"
 			(at 281.94 279.4 0)
 			(effects

Commit message: Sync
Parts:
- J3: footprint Connector_USB:USB_C_Receptacle_XKB_U262-16XN-4BVC11 -> decoder:USB_C_Receptacle_GCT_USB4800
Changed lines of the file:
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@@
 			)
 		)
-		(property "Footprint" "Connector_USB:USB_C_Receptacle_XKB_U262-16XN-4BVC11"
+		(property "Footprint" "decoder:USB_C_Receptacle_GCT_USB4800"
 			(at 308.61 76.2 0)
 			(effects

Commit message: Got FW working
Connections:
- net FIFO_EN_3V3: now also U2.5 (GPIO3), U6.6 (1A2); no longer U2.2 (GPIO1), U6.2 (1A0)
- net FIFO_R/~{W}_3V3: now also U2.2 (GPIO1), U6.2 (1A0); no longer U2.4 (GPIO2), U6.4 (1A1)
- net ~{RESET}_3V3: now also U2.4 (GPIO2), U6.4 (1A1); no longer U2.5 (GPIO3), U6.6 (1A2)
Changed lines of the file:
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@@
+		)
+	)
+	(label "~{RESET}_3V3"
+		(at 161.29 83.82 180)
+		(fields_autoplaced yes)
+		(effects
+			(font
+				(size 1.27 1.27)
+			)
+			(justify right bottom)
 		)
 	)
@@
 		)
 	)
-	(label "FIFO_R{slash}~{W}_3V3"
-		(at 309.88 175.26 0)
-		(fields_autoplaced yes)
-		(effects
-			(font
-				(size 1.27 1.27)
-			)
-			(justify left bottom)
-		)
-	)
 	(label "FIFO_EXT_D5"
 		(at 102.87 172.72 0)
@@
 		)
 	)
-	(label "FIFO_EN_3V3"
-		(at 161.29 81.28 180)
-		(fields_autoplaced yes)
-		(effects
-			(font
-				(size 1.27 1.27)
-			)
-			(justify right bottom)
-		)
-	)
 	(label "TRCVR_~{OE}"
 		(at 309.88 187.96 0)
@@
 		)
 	)
-	(label "FIFO_R{slash}~{W}_3V3"
-		(at 161.29 83.82 180)
-		(fields_autoplaced yes)
-		(effects
-			(font
-				(size 1.27 1.27)
-			)
-			(justify right bottom)
-		)
-	)
 	(label "CARD_A5"
 		(at 26.67 162.56 0)
@@
 		)
 	)
-	(label "~{RESET}_3V3"
-		(at 161.29 86.36 180)
-		(fields_autoplaced yes)
-		(effects
-			(font
-				(size 1.27 1.27)
-			)
-			(justify right bottom)
-		)
-	)
 	(label "FIFO_EXT_A0"
 		(at 82.55 152.4 180)
@@
 		)
 	)
-	(label "FIFO_EN_3V3"
-		(at 309.88 170.18 0)
-		(fields_autoplaced yes)
-		(effects
-			(font
-				(size 1.27 1.27)
-			)
-			(justify left bottom)
-		)
-	)
 	(label "FIFO_D6_3V3"
 		(at 158.75 182.88 180)
@@
 		)
 	)
+	(label "~{RESET}_3V3"
+		(at 309.88 175.26 0)
+		(fields_autoplaced yes)
+		(effects
+			(font
+				(size 1.27 1.27)
+			)
+			(justify left bottom)
+		)
+	)
 	(label "USB_D+"
 		(at 351.79 78.74 180)
@@
 		)
 	)
+	(label "FIFO_R{slash}~{W}_3V3"
+		(at 161.29 81.28 180)
+		(fields_autoplaced yes)
+		(effects
+			(font
+				(size 1.27 1.27)
+			)
+			(justify right bottom)
+		)
+	)
 	(label "FIFO_A1_3V3"
 		(at 161.29 88.9 180)
@@
 		)
 	)
-	(label "~{RESET}_3V3"
+	(label "FIFO_EN_3V3"
 		(at 309.88 177.8 0)
 		(fields_autoplaced yes)
@@
 		)
 	)
+	(label "FIFO_EN_3V3"
+		(at 161.29 86.36 180)
+		(fields_autoplaced yes)
+		(effects
+			(font
+				(size 1.27 1.27)
+			)
+			(justify right bottom)
+		)
+	)
 	(label "CARD_A1"
 		(at 68.58 64.77 180)
@@
 		)
 	)
+	(label "FIFO_R{slash}~{W}_3V3"
+		(at 309.88 170.18 0)
+		(fields_autoplaced yes)
+		(effects
+			(font
+				(size 1.27 1.27)
+			)
+			(justify left bottom)
+		)
+	)
